Commit message: update object  point cloud and normals getting

File: assets/maze.urdf (robot description, URDF)
Before this commit: robot maze, 141 links, 140 joints
Links:
- removed link block_9_6
- added link block_7_6, mass 0; collision box size=1.0 1.0 2.0; visual box size=1.0 1.0 2.0
Joints:
- removed joint joint_block_9_6
- added joint joint_block_7_6: type fixed, parent maze_base, child block_7_6, origin xyz=2.5 -1.5 1.0 rpy=0 0 0
