Commit message: update env & keyboard controller

File: assets/fetch/fetch.urdf (robot description, URDF)
Before this commit: robot fetch, 29 links, 28 joints
Links:
- link base_link: geometry collision mesh filename=fetch_description/meshes/base_link_collision.STL; visual mesh filename=fetch_description/meshes/base_link.obj
- link elbow_flex_link: geometry collision mesh filename=fetch_description/meshes/elbow_flex_link_collision.STL; visual mesh filename=fetch_description/meshes/elbow_flex_link.obj
- link estop_link: geometry collision mesh filename=fetch_description/meshes/estop_link.STL; visual mesh filename=fetch_description/meshes/estop_link.obj
- link forearm_roll_link: geometry collision mesh filename=fetch_description/meshes/forearm_roll_link_collision.STL; visual mesh filename=fetch_description/meshes/forearm_roll_link.obj
- link gripper_link: geometry collision mesh filename=fetch_description/meshes/gripper_link.STL; visual mesh filename=fetch_description/meshes/gripper_link.obj
- link head_pan_link: geometry collision mesh filename=fetch_description/meshes/head_pan_link_collision.STL; visual mesh filename=fetch_description/meshes/head_pan_link.obj
- link head_tilt_link: geometry collision mesh filename=fetch_description/meshes/head_tilt_link_collision.STL; visual mesh filename=fetch_description/meshes/head_tilt_link.obj
- link shoulder_lift_link: geometry collision mesh filename=fetch_description/meshes/shoulder_lift_link_collision.STL; visual mesh filename=fetch_description/meshes/shoulder_lift_link.obj
- link shoulder_pan_link: geometry collision mesh filename=fetch_description/meshes/shoulder_pan_link_collision.STL; visual mesh filename=fetch_description/meshes/shoulder_pan_link.obj
- link torso_fixed_link: geometry collision mesh filename=fetch_description/meshes/torso_fixed_link.STL; visual mesh filename=fetch_description/meshes/torso_fixed_link.obj
- link torso_lift_link: geometry collision mesh filename=fetch_description/meshes/torso_lift_link_collision.STL; visual mesh filename=fetch_description/meshes/torso_lift_link.obj
- link upperarm_roll_link: geometry collision mesh filename=fetch_description/meshes/upperarm_roll_link_collision.STL; visual mesh filename=fetch_description/meshes/upperarm_roll_link.obj
- link wrist_flex_link: geometry collision mesh filename=fetch_description/meshes/wrist_flex_link_collision.STL; visual mesh filename=fetch_description/meshes/wrist_flex_link.obj
- link wrist_roll_link: geometry collision mesh filename=fetch_description/meshes/wrist_roll_link_collision.STL; visual mesh filename=fetch_description/meshes/wrist_roll_link.obj

Commit message: update gripper collision

File: assets/fetch/fetch.urdf (robot description, URDF)
Before this commit: robot fetch, 29 links, 28 joints
Links:
- link l_gripper_finger_link: geometry collision box size=0.063 0.012 0.024; visual mesh filename=fetch_description/meshes/l_gripper_finger_link.STL
- link r_gripper_finger_link: geometry collision box size=0.063 0.012 0.024; visual mesh filename=fetch_description/meshes/r_gripper_finger_link.STL
